Commit message: Modify URDF

File: rr_openrover_description/urdf/4WD_rover.urdf.xacro (robot description, xacro)
@@ -2,10 +2,9 @@
 <robot name="2WD_rover" xmlns:xacro="http://ros.org/wiki/xacro">
   <xacro:include filename="$(find rr_openrover_description)/urdf/common_properties.xacro"/>
-  <xacro:include filename="$(find rr_openrover_description)/urdf/4WD_Rover.gazebo.xacro"/>
   <link name="base_footprint"/>
   <joint name="base_joint" type="fixed">
     <parent link="base_footprint"/>
     <child link="base_link"/>
-    <origin xyz="0 0 0.12" rpy="0 0 0"/>
+    <origin xyz="0 0 0" rpy="0 0 0"/>
   </joint>
   <link name="base_link">
@@ -40,5 +39,5 @@
       <origin xyz="0 0 0" rpy="0 0 0"/>
       <geometry>
-        <box size="0.32 0.175 0.005"/>
+        <box size="0.305 0.178 0.005"/>
       </geometry>
       <material name="light_black"/>
@@ -55,11 +54,11 @@
     <parent link="bottom_plate_link"/>
     <child link="xavier_link"/>
-    <origin xyz="-0.0032 0 0.0275" rpy="0 0 0"/>
+    <origin xyz="-0.0832 0 0.0275" rpy="0 0 0"/>
   </joint>
   <link name="xavier_link">
     <visual>
-      <origin xyz="-0.08 0 0" rpy="0 0 0"/>
+      <origin xyz="0 0 0" rpy="0 0 0"/>
       <geometry>
-        <box size="0.111 0.117 0.05"/>
+        <box size="0.105 0.092 0.065"/>
       </geometry>
       <material name="light_black"/>
@@ -76,5 +75,5 @@
     <parent link="bottom_plate_link"/>
     <child link="top_plate_link"/>
-    <origin xyz="0 0 0.1" rpy="0 0 0"/>
+    <origin xyz="0 0 0.12" rpy="0 0 0"/>
   </joint>
   <link name="top_plate_link">
@@ -93,4 +92,18 @@
                ixz="0.0" iyz="0.0" izz="1.136e-2" />
     </inertial>
+  </link>
+  <joint name="realsense_link_joint" type="fixed">
+    <parent link="top_plate_link"/>
+    <child link="realsense_link"/>
+    <origin xyz="0.145 0 -0.0125" rpy="0 0 0"/>
+  </joint>
+  <link name="realsense_link">
+    <visual>
+      <origin xyz="0 0 0" rpy="0 0 0"/>
+      <geometry>
+        <box size="0.025 0.089 0.025"/>
+      </geometry>
+      <material name="grey"/>
+    </visual>
   </link>
   <joint name="lidar_link_joint" type="fixed">
@@ -115,3 +128,59 @@
     </inertial>
   </link>
+  <joint name="standoff_fl_joint" type="fixed">
+    <parent link="bottom_plate_link"/>
+    <child link="standoff_fl_link"/>
+    <origin xyz="0.14 -0.074 0.0025" rpy="0 0 0"/>
+  </joint>
+  <link name="standoff_fl_link">
+    <visual>
+      <origin xyz="0 0 0.06" rpy="0 0 0"/>
+      <geometry>
+        <cylinder length="0.12" radius="0.0043"/>
+      </geometry>
+      <material name="grey"/>
+    </visual>
+  </link>
+  <joint name="standoff_fr_link_joint" type="fixed">
+    <parent link="bottom_plate_link"/>
+    <child link="standoff_fr_link"/>
+    <origin xyz="0.14 0.074 0.0025" rpy="0 0 0"/>
+  </joint>
+  <link name="standoff_fr_link">
+    <visual>
+      <origin xyz="0 0 0.06" rpy="0 0 0"/>
+      <geometry>
+        <cylinder length="0.12" radius="0.0043"/>
+      </geometry>
+      <material name="grey"/>
+    </visual>
+  </link>
+  <joint name="standoff_bl_link_joint" type="fixed">
+    <parent link="bottom_plate_link"/>
+    <child link="standoff_bl_link"/>
+    <origin xyz="-0.14 -0.074 0.0025" rpy="0 0 0"/>
+  </joint>
+  <link name="standoff_bl_link">
+    <visual>
+      <origin xyz="0 0 0.06" rpy="0 0 0"/>
+      <geometry>
+        <cylinder length="0.12" radius="0.0043"/>
+      </geometry>
+      <material name="grey"/>
+    </visual>
+  </link>
+  <joint name="standoff_br_link_joint" type="fixed">
+    <parent link="bottom_plate_link"/>
+    <child link="standoff_br_link"/>
+    <origin xyz="-0.14 0.074 0.0025" rpy="0 0 0"/>
+  </joint>
+  <link name="standoff_br_link">
+    <visual>
+      <origin xyz="0 0 0.06" rpy="0 0 0"/>
+      <geometry>
+        <cylinder length="0.12" radius="0.0043"/>
+      </geometry>
+      <material name="grey"/>
+    </visual>
+  </link>
 </robot>

Commit message: Split apart chassis and SLAM pack into separate files

File: rr_openrover_description/urdf/4WD_rover.urdf.xacro (robot description, xacro)
@@ -1,14 +1,16 @@
 <?xml version="1.0" ?>
-<robot name="2WD_rover" xmlns:xacro="http://ros.org/wiki/xacro">
+<robot name="4WD_rover" xmlns:xacro="http://ros.org/wiki/xacro">
   <xacro:include filename="$(find rr_openrover_description)/urdf/common_properties.xacro"/>
-  <link name="base_footprint"/>
-  <joint name="base_joint" type="fixed">
-    <parent link="base_footprint"/>
-    <child link="base_link"/>
+  <xacro:property name="PI" value="3.1415926535897931" />
+  <xacro:property name="rover_4wd_ground_clearance" value="0.182" />
+  <link name="base_link"/>
+  <joint name="base_link_joint" type="fixed">
+    <parent link="base_link"/>
+    <child link="chassis_link"/>
     <origin xyz="0 0 0" rpy="0 0 0"/>
   </joint>
-  <link name="base_link">
+  <link name="chassis_link">
     <visual>
-      <origin xyz="0 0 0.182" rpy="0 0 1.57"/>
+      <origin xyz="0 0 ${rover_4wd_ground_clearance}" rpy="0 0 ${PI/2}"/>
       <geometry>
         <mesh filename="package://rr_openrover_description/meshes/4WD_OpenRover.stl" scale="1 1 1"/>
@@ -30,157 +32,4 @@
     </inertial>
   </link>
-  <joint name="bottom_plate_link_joint" type="fixed">
-    <parent link="base_link"/>
-    <child link="bottom_plate_link"/>
-    <origin xyz="0.025 0 0.185" rpy="0 0 0"/>
-  </joint>
-  <link name="bottom_plate_link">
-    <visual>
-      <origin xyz="0 0 0" rpy="0 0 0"/>
-      <geometry>
-        <box size="0.305 0.178 0.005"/>
-      </geometry>
-      <material name="light_black"/>
-    </visual>
-    <inertial>
-      <origin xyz="0 0 0" />
-      <mass value="0.65" />
-      <inertia ixx="3.496e-3"
-               ixy="0.0" iyy="7.864e-3"
-               ixz="0.0" iyz="0.0" izz="1.136e-2" />
-    </inertial>
-  </link>
-  <joint name="xavier_link_joint" type="fixed">
-    <parent link="bottom_plate_link"/>
-    <child link="xavier_link"/>
-    <origin xyz="-0.0832 0 0.0275" rpy="0 0 0"/>
-  </joint>
-  <link name="xavier_link">
-    <visual>
-      <origin xyz="0 0 0" rpy="0 0 0"/>
-      <geometry>
-        <box size="0.105 0.092 0.065"/>
-      </geometry>
-      <material name="light_black"/>
-    </visual>
-    <inertial>
-      <origin xyz="0 0 0" />
-      <mass value="0.64" />
-      <inertia ixx="8.634e-4"
-               ixy="0.0" iyy="7.905e-4"
-               ixz="0.0" iyz="0.0" izz="1.387e-3" />
-    </inertial>
-  </link>
-  <joint name="top_plate_link_joint" type="fixed">
-    <parent link="bottom_plate_link"/>
-    <child link="top_plate_link"/>
-    <origin xyz="0 0 0.12" rpy="0 0 0"/>
-  </joint>
-  <link name="top_plate_link">
-    <visual>
-      <origin xyz="0 0 0" rpy="0 0 0"/>
-      <geometry>
-        <box size="0.32 0.175 0.005"/>
-      </geometry>
-      <material name="light_black"/>
-    </visual>
-    <inertial>
-      <origin xyz="0 0 0" />
-      <mass value="0.65" />
-      <inertia ixx="3.496e-3"
-               ixy="0.0" iyy="7.864e-3"
-               ixz="0.0" iyz="0.0" izz="1.136e-2" />
-    </inertial>
-  </link>
-  <joint name="realsense_link_joint" type="fixed">
-    <parent link="top_plate_link"/>
-    <child link="realsense_link"/>
-    <origin xyz="0.145 0 -0.0125" rpy="0 0 0"/>
-  </joint>
-  <link name="realsense_link">
-    <visual>
-      <origin xyz="0 0 0" rpy="0 0 0"/>
-      <geometry>
-        <box size="0.025 0.089 0.025"/>
-      </geometry>
-      <material name="grey"/>
-    </visual>
-  </link>
-  <joint name="lidar_link_joint" type="fixed">
-    <parent link="top_plate_link"/>
-    <child link="lidar_link"/>
-    <origin xyz="0.105 0 0.02" rpy="0 0 0"/>
-  </joint>
-  <link name="lidar_link">
-    <visual>
-      <origin xyz="0 0 0" rpy="0 0 0"/>
-      <geometry>
-        <cylinder length="0.04" radius="0.03"/>
-      </geometry>
-      <material name="light_black"/>
-    </visual>
-    <inertial>
-      <origin xyz="0 0 0" />
-      <mass value="0.220" />
-      <inertia ixx="1.214e-4"
-               ixy="0.0" iyy="1.214e-4"
-               ixz="0.0" iyz="0.0" izz="1.597e-4" />
-    </inertial>
-  </link>
-  <joint name="standoff_fl_joint" type="fixed">
-    <parent link="bottom_plate_link"/>
-    <child link="standoff_fl_link"/>
-    <origin xyz="0.14 -0.074 0.0025" rpy="0 0 0"/>
-  </joint>
-  <link name="standoff_fl_link">
-    <visual>
-      <origin xyz="0 0 0.06" rpy="0 0 0"/>
-      <geometry>
-        <cylinder length="0.12" radius="0.0043"/>
-      </geometry>
-      <material name="grey"/>
-    </visual>
-  </link>
-  <joint name="standoff_fr_link_joint" type="fixed">
-    <parent link="bottom_plate_link"/>
-    <child link="standoff_fr_link"/>
-    <origin xyz="0.14 0.074 0.0025" rpy="0 0 0"/>
-  </joint>
-  <link name="standoff_fr_link">
-    <visual>
-      <origin xyz="0 0 0.06" rpy="0 0 0"/>
-      <geometry>
-        <cylinder length="0.12" radius="0.0043"/>
-      </geometry>
-      <material name="grey"/>
-    </visual>
-  </link>
-  <joint name="standoff_bl_link_joint" type="fixed">
-    <parent link="bottom_plate_link"/>
-    <child link="standoff_bl_link"/>
-    <origin xyz="-0.14 -0.074 0.0025" rpy="0 0 0"/>
-  </joint>
-  <link name="standoff_bl_link">
-    <visual>
-      <origin xyz="0 0 0.06" rpy="0 0 0"/>
-      <geometry>
-        <cylinder length="0.12" radius="0.0043"/>
-      </geometry>
-      <material name="grey"/>
-    </visual>
-  </link>
-  <joint name="standoff_br_link_joint" type="fixed">
-    <parent link="bottom_plate_link"/>
-    <child link="standoff_br_link"/>
-    <origin xyz="-0.14 0.074 0.0025" rpy="0 0 0"/>
-  </joint>
-  <link name="standoff_br_link">
-    <visual>
-      <origin xyz="0 0 0.06" rpy="0 0 0"/>
-      <geometry>
-        <cylinder length="0.12" radius="0.0043"/>
-      </geometry>
-      <material name="grey"/>
-    </visual>
-  </link>
+<xacro:include filename="$(find rr_openrover_description)/urdf/accessories.urdf.xacro" />
 </robot>
